File: hardware/Boelgene_v1/Boelgene_v1.kicad_pcb (KiCad board)
At the start: 2 copper layers, 65 parts, among them J1 batt, J2 pressure3, J3 pressure2, J4 pressure1, J5 pressure4, U1 Pico, U2 MCP3008, U3 PT8211-pt8211

Commit message: Routing of pcb
Parts:
- added C10: 1u dac2, Capacitor_THT:CP_Radial_D5.0mm_P2.50mm, F.Cu at (88.0, 112.3)
- added C11: 1u dac1, Capacitor_THT:CP_Radial_D5.0mm_P2.50mm, F.Cu at (96.4, 119.8)
- added C12: 1u dac2, Capacitor_THT:CP_Radial_D5.0mm_P2.50mm, F.Cu at (96.2, 112.3)
- added C7: 1u pwm, Capacitor_THT:CP_Radial_D5.0mm_P2.50mm, F.Cu at (37.1, 97.0)
- added C8: 1u pwm, Capacitor_THT:CP_Radial_D5.0mm_P2.50mm, F.Cu at (45.2, 97.0)
- added C9: 1u dac1, Capacitor_THT:CP_Radial_D5.0mm_P2.50mm, F.Cu at (87.7, 119.9)
- C2, C4: footprint Capacitor_THT:CP_Radial_D10.0mm_P3.80mm -> Capacitor_THT:CP_Radial_D8.0mm_P5.00mm
- moved J1 100.3 mm to (106.4, 114.8)
- moved TP4 92.1 mm to (53.3, 86.4)
- moved TP11 88.4 mm to (48.3, 83.8)
- moved TP2 84.2 mm to (48.3, 86.4)
- moved TP3 83.9 mm to (50.8, 83.8)
- moved TP10 82.2 mm to (50.8, 86.4)
- moved TP6 82.1 mm to (110.2, 107.7)
- moved TP9 81.8 mm to (53.3, 83.8)
- moved TP12 80.7 mm to (105.2, 105.2)
- moved TP1 78.6 mm to (107.7, 105.2)
- moved TP5 77.6 mm to (110.2, 105.2)
- moved TP7 73.7 mm to (105.2, 107.7)
- moved TP8 71.4 mm to (107.7, 107.7)
- moved TP28 70.5 mm to (57.9, 97.0)
- moved TP26 63.5 mm to (44.7, 82.3)
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Connections:
- TP43 pad 1: Net-(U1-Pad1) -> Net-(TP43-Pad1)
- TP44 pad 1: LCH -> Net-(TP44-Pad1)
- TP45 pad 1: RCH -> Net-(TP45-Pad1)
Routing:
- net filtered_3.3: track 0.00 -> 181.5 mm
- net GND: track 0.00 -> 174.6 mm
- net GNDA: track 0.00 -> 159.3 mm
- net batt+: track 0.00 -> 113.5 mm
- net +3.3V: track 0.00 -> 107.6 mm, vias 0 -> 2
- net filtered_vcc: track 0.00 -> 42.3 mm
- net Net-(U1-Pad1): track 0.00 -> 42.2 mm
- net Net-(U1-Pad24): track 0.00 -> 34.5 mm
- net Net-(U1-Pad22): track 0.00 -> 34.4 mm
- net LCH: track 0.00 -> 25.2 mm
- net RCH: track 0.00 -> 24.3 mm
- net Net-(U1-Pad21): track 0.00 -> 22.2 mm
- net Net-(J5-Pad2): track 0.00 -> 20.8 mm
- net Net-(J3-Pad2): track 0.00 -> 19.9 mm
- net Net-(J2-Pad2): track 0.00 -> 19.5 mm
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- added copper zone on F.Cu, net GNDA

Commit message: Updated PCB
Parts:
- added G***: LOGO, PCB_symbols:owl_7x10, F.Cu at (105.2, 126.0)
- added H1: MountingHole, MountingHole:MountingHole_3.2mm_M3, F.Cu at (31.5, 81.3)
- added H2: MountingHole, MountingHole:MountingHole_3.2mm_M3, F.Cu at (31.5, 128.0)
- added H3: MountingHole, MountingHole:MountingHole_3.2mm_M3, F.Cu at (111.8, 81.3)
- added H4: MountingHole, MountingHole:MountingHole_3.2mm_M3, F.Cu at (111.8, 127.5)
- C6: footprint Capacitor_THT:CP_Radial_D4.0mm_P2.00mm -> Capacitor_THT:CP_Radial_D5.0mm_P2.00mm
- TP1, TP10, TP11, TP12, TP13, TP14, TP15, TP16, TP17, TP18, TP19, TP2, TP20, TP21, TP22, TP23, TP24, TP25, TP26, TP27, TP28, TP29, TP3, TP30, TP31, TP32, TP33, TP34, TP35, TP36, TP37, TP38, TP39, TP4, TP40, TP41, TP42, TP43, TP44, TP45, TP5, TP6, TP7, TP8, TP9: footprint TestPoint:TestPoint_THTPad_1.5x1.5mm_Drill0.7mm -> TestPoint:TestPoint_THTPad_2.0x2.0mm_Drill1.0mm
- moved TP41 4.06 mm to (106.2, 81.8)
- moved RV4 3.10 mm to (107.7, 95.5)
- moved TP20 2.54 mm to (65.0, 126.5)
- moved J5 2.54 mm to (111.8, 90.4)
- moved TP32 2.27 mm to (56.9, 81.8)
- moved TP13 2.03 mm to (40.1, 126.5)
- moved TP33 1.76 mm to (59.9, 81.8)
- moved TP19 1.52 mm to (61.5, 126.5)
- moved TP39 1.28 mm to (78.2, 81.8)
- moved TP34 1.26 mm to (63.0, 81.8)
- moved TP14 1.02 mm to (43.7, 126.5)
- moved TP16 1.02 mm to (50.8, 126.5)
- moved TP38 0.78 mm to (75.2, 81.8)
- moved TP35 0.75 mm to (66.0, 81.8)
- moved TP17 0.51 mm to (54.4, 126.5)
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Routing:
- net Net-(J5-Pad2): track 20.8 -> 25.2 mm
- net GNDA: track 159.3 -> 156.4 mm
- net batt+: track 113.5 -> 116.3 mm
- net Net-(TP32-Pad1): track 3.31 -> 5.43 mm
- net GND: track 174.6 -> 176.5 mm
- net Net-(TP20-Pad1): track 5.44 -> 6.28 mm
- net Net-(TP13-Pad1): track 5.44 -> 6.28 mm
- net Net-(TP33-Pad1): track 3.31 -> 4.04 mm
- net Net-(TP19-Pad1): track 5.44 -> 6.07 mm
- net Net-(U1-Pad21): track 22.2 -> 22.8 mm
- net Net-(TP16-Pad1): track 5.44 -> 6.01 mm
- net Net-(TP39-Pad1): track 3.31 -> 3.85 mm
- net Net-(TP34-Pad1): track 3.31 -> 3.83 mm
Other:
- board text added: "Raspberry Pico - RP2040"
- board text added: "TES - Bølgene v1 Handmade in Norway"
