File: hardware/Boelgene_v1/Boelgene_v1.kicad_sch (KiCad schematic)
At the start: 6 parts, among them U1 Pico, U2 MCP3008

Commit message: Updated sch
Parts:
- added C?: 1u, symbol Device:C_Polarized
Connections:
- net +3.3V: now also C?.1
- net GNDA: now also C?.2
Changed lines of the file:
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@@
   (junction (at 150.114 61.214) (diameter 0) (color 0 0 0 0)
   )
+  (junction (at 214.122 87.884) (diameter 0) (color 0 0 0 0)
+  )
   (wire (pts (xy 166.878 56.388) (xy 166.878 65.024))
     (stroke (width 0) (type default) (color 0 0 0 0))
@@
     (stroke (width 0) (type default) (color 0 0 0 0))
   )
+  (wire (pts (xy 214.122 87.884) (xy 214.122 80.01))
+    (stroke (width 0) (type default) (color 0 0 0 0))
+  )
   (wire (pts (xy 170.688 64.77) (xy 203.962 64.77))
     (stroke (width 0) (type default) (color 0 0 0 0))
@@
     (stroke (width 0) (type default) (color 0 0 0 0))
   )
+  (wire (pts (xy 214.122 89.916) (xy 214.122 87.884))
+    (stroke (width 0) (type default) (color 0 0 0 0))
+  )
   (wire (pts (xy 164.084 56.388) (xy 166.878 56.388))
     (stroke (width 0) (type default) (color 0 0 0 0))
@@
   )
   (wire (pts (xy 175.768 67.31) (xy 175.768 104.394))
+    (stroke (width 0) (type default) (color 0 0 0 0))
+  )
+  (wire (pts (xy 206.502 87.884) (xy 206.502 90.932))
     (stroke (width 0) (type default) (color 0 0 0 0))
   )
@@
     )
   )
-  (symbol (lib_id "power:+3.3V") (at 214.122 80.01 180) (unit 1)
-    (in_bom yes) (on_board yes) (fields_autoplaced)
-    (property "Reference" "#PWR05" (id 0) (at 214.122 76.2 0)
-      (effects (font (size 1.27 1.27)) hide)
-    )
-    (property "Value" "+3.3V" (id 1) (at 214.122 84.4534 0))
-    (property "Footprint" "" (id 2) (at 214.122 80.01 0)
-      (effects (font (size 1.27 1.27)) hide)
-    )
-    (property "Datasheet" "" (id 3) (at 214.122 80.01 0)
+  (symbol (lib_id "power:+3.3V") (at 214.122 89.916 180) (unit 1)
+    (in_bom yes) (on_board yes) (fields_autoplaced)
+    (property "Reference" "#PWR05" (id 0) (at 214.122 86.106 0)
+      (effects (font (size 1.27 1.27)) hide)
+    )
+    (property "Value" "+3.3V" (id 1) (at 214.122 94.3594 0))
+    (property "Footprint" "" (id 2) (at 214.122 89.916 0)
+      (effects (font (size 1.27 1.27)) hide)
+    )
+    (property "Datasheet" "" (id 3) (at 214.122 89.916 0)
       (effects (font (size 1.27 1.27)) hide)
     )
@@
     )
     (pin "1")
+  )
+  (symbol (lib_id "Device:C_Polarized") (at 210.312 87.884 270) (unit 1)
+    (in_bom yes) (on_board yes) (fields_autoplaced)
+    (property "Reference" "C?" (id 0) (at 211.201 82.0252 90))
+    (property "Value" "1u" (id 1) (at 211.201 84.5621 90))
+    (property "Footprint" "" (id 2) (at 206.502 88.8492 0)
+      (effects (font (size 1.27 1.27)) hide)
+    )
+    (property "Datasheet" "~" (id 3) (at 210.312 87.884 0)
+      (effects (font (size 1.27 1.27)) hide)
+    )
+    (pin "1")
+    (pin "2")
   )
   (symbol (lib_id "Device:R") (at 198.12 35.052 90) (unit 1)
@@
     (pin "9")
   )
+  (symbol (lib_id "power:GNDA") (at 206.502 90.932 0) (unit 1)
+    (in_bom yes) (on_board yes) (fields_autoplaced)
+    (property "Reference" "#PWR?" (id 0) (at 206.502 97.282 0)
+      (effects (font (size 1.27 1.27)) hide)
+    )
+    (property "Value" "GNDA" (id 1) (at 206.502 95.3754 0))
+    (property "Footprint" "" (id 2) (at 206.502 90.932 0)
+      (effects (font (size 1.27 1.27)) hide)
+    )
+    (property "Datasheet" "" (id 3) (at 206.502 90.932 0)
+      (effects (font (size 1.27 1.27)) hide)
+    )
+    (pin "1")
+  )
   (symbol (lib_id "power:GNDA") (at 217.932 49.276 180) (unit 1)
     (in_bom yes) (on_board yes) (fields_autoplaced)
@@
       (reference "#PWR06") (unit 1) (value "GNDA") (footprint "")
     )
+    (path "/def93be6-0264-4192-8e6a-813f8a290a83"
+      (reference "#PWR?") (unit 1) (value "GNDA") (footprint "")
+    )
     (path "/573556f2-90b0-4009-b88c-7c1cf8ebccda"
       (reference "C1") (unit 1) (value "0.1u") (footprint "")
@@
       (reference "C3") (unit 1) (value "100n") (footprint "Capacitor_THT:C_Axial_L3.8mm_D2.6mm_P7.50mm_Horizontal")
     )
+    (path "/352509e3-4e18-45a3-83d6-b5e6dd362b91"
+      (reference "C?") (unit 1) (value "1u") (footprint "")
+    )
     (path "/546471a4-25fa-41f4-baaf-788a86c152b6"

Commit message: Added kicad components
Parts:
- added C4: 100u, Capacitor_THT:CP_Radial_D10.0mm_P3.80mm, symbol Device:C_Polarized
- added C5: 100n, Capacitor_THT:C_Axial_L3.8mm_D2.6mm_P7.50mm_Horizontal, symbol Device:C
- added J1: batt, Connector_JST:JST_XH_B2B-XH-A_1x02_P2.50mm_Vertical, symbol Connector:Conn_01x02_Female
- added J2: pressure3, Connector_JST:JST_XH_B2B-XH-A_1x02_P2.50mm_Vertical, symbol Connector:Conn_01x02_Female
- added J3: pressure2, Connector_JST:JST_XH_B2B-XH-A_1x02_P2.50mm_Vertical, symbol Connector:Conn_01x02_Female
- added J4: pressure1, Connector_JST:JST_XH_B2B-XH-A_1x02_P2.50mm_Vertical, symbol Connector:Conn_01x02_Female
- added J5: pressure4, Connector_JST:JST_XH_B2B-XH-A_1x02_P2.50mm_Vertical, symbol Connector:Conn_01x02_Female
- added R2: 10, Resistor_THT:R_Axial_DIN0207_L6.3mm_D2.5mm_P7.62mm_Horizontal, symbol Device:R
- added RV1: 20k_adj3, Potentiometer_THT:Potentiometer_Runtron_RM-065_Vertical, symbol Device:R_Potentiometer
- added RV2: 20k_adj2, Potentiometer_THT:Potentiometer_Runtron_RM-065_Vertical, symbol Device:R_Potentiometer
- added RV3: 20k_adj1, Potentiometer_THT:Potentiometer_Runtron_RM-065_Vertical, symbol Device:R_Potentiometer
- added RV4: 20k_adj4, Potentiometer_THT:Potentiometer_Runtron_RM-065_Vertical, symbol Device:R_Potentiometer
- added TP1, TP12, TP5, TP6, TP7, TP8: GND, TestPoint:TestPoint_THTPad_1.5x1.5mm_Drill0.7mm, symbol Connector:TestPoint
- added TP10, TP11, TP2, TP3, TP4, TP9: ADC_ref, TestPoint:TestPoint_THTPad_1.5x1.5mm_Drill0.7mm, symbol Connector:TestPoint
- added TP13: D2, TestPoint:TestPoint_THTPad_1.5x1.5mm_Drill0.7mm, symbol Connector:TestPoint
- added TP14: D3, TestPoint:TestPoint_THTPad_1.5x1.5mm_Drill0.7mm, symbol Connector:TestPoint
- added TP15: D4, TestPoint:TestPoint_THTPad_1.5x1.5mm_Drill0.7mm, symbol Connector:TestPoint
- added TP16: D5, TestPoint:TestPoint_THTPad_1.5x1.5mm_Drill0.7mm, symbol Connector:TestPoint
- added TP17: D6, TestPoint:TestPoint_THTPad_1.5x1.5mm_Drill0.7mm, symbol Connector:TestPoint
- added TP18: D7, TestPoint:TestPoint_THTPad_1.5x1.5mm_Drill0.7mm, symbol Connector:TestPoint
- added TP19: D8, TestPoint:TestPoint_THTPad_1.5x1.5mm_Drill0.7mm, symbol Connector:TestPoint
- added TP20: D9, TestPoint:TestPoint_THTPad_1.5x1.5mm_Drill0.7mm, symbol Connector:TestPoint
- added TP21, TP22, TP23, TP24, TP25, TP26: GNDA, TestPoint:TestPoint_THTPad_1.5x1.5mm_Drill0.7mm, symbol Connector:TestPoint
- added TP27: AI28, TestPoint:TestPoint_THTPad_1.5x1.5mm_Drill0.7mm, symbol Connector:TestPoint
- added TP28: AI27, TestPoint:TestPoint_THTPad_1.5x1.5mm_Drill0.7mm, symbol Connector:TestPoint
- added TP29: AI26, TestPoint:TestPoint_THTPad_1.5x1.5mm_Drill0.7mm, symbol Connector:TestPoint
- added TP30: pressure3_out, TestPoint:TestPoint_THTPad_1.5x1.5mm_Drill0.7mm, symbol Connector:TestPoint
- added TP31: pressure2_out, TestPoint:TestPoint_THTPad_1.5x1.5mm_Drill0.7mm, symbol Connector:TestPoint
- added TP32: adc7, TestPoint:TestPoint_THTPad_1.5x1.5mm_Drill0.7mm, symbol Connector:TestPoint
- added TP33: adc6, TestPoint:TestPoint_THTPad_1.5x1.5mm_Drill0.7mm, symbol Connector:TestPoint
- added TP34: adc5, TestPoint:TestPoint_THTPad_1.5x1.5mm_Drill0.7mm, symbol Connector:TestPoint
- added TP35: adc4, TestPoint:TestPoint_THTPad_1.5x1.5mm_Drill0.7mm, symbol Connector:TestPoint
- added TP36: adc3, TestPoint:TestPoint_THTPad_1.5x1.5mm_Drill0.7mm, symbol Connector:TestPoint
- added TP37: adc2, TestPoint:TestPoint_THTPad_1.5x1.5mm_Drill0.7mm, symbol Connector:TestPoint
- added TP38: adc1, TestPoint:TestPoint_THTPad_1.5x1.5mm_Drill0.7mm, symbol Connector:TestPoint
- added TP39: adc0, TestPoint:TestPoint_THTPad_1.5x1.5mm_Drill0.7mm, symbol Connector:TestPoint
- added TP40: pressure1_out, TestPoint:TestPoint_THTPad_1.5x1.5mm_Drill0.7mm, symbol Connector:TestPoint
- added TP41: pressure4_out, TestPoint:TestPoint_THTPad_1.5x1.5mm_Drill0.7mm, symbol Connector:TestPoint
- added TP42: 3.3V, TestPoint:TestPoint_THTPad_1.5x1.5mm_Drill0.7mm, symbol Connector:TestPoint
- added TP43: out_PWM, TestPoint:TestPoint_THTPad_1.5x1.5mm_Drill0.7mm, symbol Connector:TestPoint
- added TP44: out_dac1, TestPoint:TestPoint_THTPad_1.5x1.5mm_Drill0.7mm, symbol Connector:TestPoint
- added TP45: out_dac2, TestPoint:TestPoint_THTPad_1.5x1.5mm_Drill0.7mm, symbol Connector:TestPoint
- added U3: PT8211-pt8211, Package_SO:SOP-8_3.9x4.9mm_P1.27mm, symbol pt8211-pt8211:PT8211-pt8211
- C1: footprint (none) -> Capacitor_THT:C_Axial_L3.8mm_D2.6mm_P7.50mm_Horizontal
- C6: renamed from C?; footprint (none) -> Capacitor_THT:CP_Radial_D4.0mm_P2.00mm
- U1: footprint RPi_Pico:RPi_Pico_SMD_TH -> Pico:RPi_Pico_SMD_TH
- U2: footprint (none) -> Package_DIP:DIP-16_W7.62mm
Connections:
- net +3.3V: now also C1.2, R2.2, TP42.1; no longer C1.1
- net GND: now also C1.1, J1.1 (Pin_1), TP1.1, TP12.1, TP5.1, TP6.1, TP7.1, TP8.1; no longer C1.2
- net GNDA: now also C4.2, C5.2, RV1.1, RV2.1, RV3.1, RV4.1, TP21.1, TP22.1, TP23.1, TP24.1, TP25.1, TP26.1, U3.4 (GND)
- net batt+: now also J1.2 (Pin_2)
- net filtered_vcc: now also U3.5 (VDD); no longer U1.35 (ADC_VREF), U2.15 (Vref)
- net at U1.1 (GPIO0): now also TP43.1
- net at U1.10 (GPIO7): now also TP18.1
- net at U1.11 (GPIO8): now also TP19.1
- net at U1.12 (GPIO9): now also TP20.1
- net at U1.26 (GPIO20): now also U3.1 (BCK)
- net at U1.27 (GPIO21): now also U3.2 (WS)
- net at U1.29 (GPIO22): now also U3.3 (DIN)
- net at U1.31 (GPIO26_ADC0): now also TP29.1
- net at U1.32 (GPIO27_ADC1): now also TP28.1
- net at U1.34 (GPIO28_ADC2): now also TP27.1
- net at U1.4 (GPIO2): now also TP13.1
- net at U1.5 (GPIO3): now also TP14.1
- net at U1.6 (GPIO4): now also TP15.1
- net at U1.7 (GPIO5): now also TP16.1
- net at U1.9 (GPIO6): now also TP17.1
- net at U2.1 (CH0): now also TP39.1
- net at U2.2 (CH1): now also TP38.1
- net at U2.3 (CH2): now also TP37.1
- net at U2.4 (CH3): now also TP36.1
- net at U2.5 (CH4): now also TP35.1
- net at U2.6 (CH5): now also TP34.1
- net at U2.7 (CH6): now also TP33.1
- net at U2.8 (CH7): now also TP32.1
- new net: J3.2 (Pin_2), RV2.2, RV2.3, TP31.1
- new net: J4.2 (Pin_2), RV3.2, RV3.3, TP40.1
- new net: J2.2 (Pin_2), RV1.2, RV1.3, TP30.1
- new net: J5.2 (Pin_2), RV4.2, RV4.3, TP41.1
- new net LCH: TP44.1, U3.6 (LCH)
- new net RCH: TP45.1, U3.8 (RCH)
- new net filtered_3.3: C4.1, C5.1, J2.1 (Pin_1), J3.1 (Pin_1), J4.1 (Pin_1), J5.1 (Pin_1), R2.1, TP10.1, TP11.1, TP2.1, TP3.1, TP4.1, TP9.1, U1.35 (ADC_VREF), U2.15 (Vref)
- no-connect marks 0 -> 19
Other:
- moved on the sheet: C1, C2, C3, R1, U1

Commit message: Routing of pcb
Parts:
- added C10, C12: 1u dac2, Capacitor_THT:CP_Radial_D5.0mm_P2.50mm, symbol Device:C_Polarized
- added C11, C9: 1u dac1, Capacitor_THT:CP_Radial_D5.0mm_P2.50mm, symbol Device:C_Polarized
- added C7, C8: 1u pwm, Capacitor_THT:CP_Radial_D5.0mm_P2.50mm, symbol Device:C_Polarized
- C2, C4: footprint Capacitor_THT:CP_Radial_D10.0mm_P3.80mm -> Capacitor_THT:CP_Radial_D8.0mm_P5.00mm
Connections:
- net LCH: now also C9.1; no longer TP44.1
- net RCH: now also C10.1; no longer TP45.1
- net at U1.1 (GPIO0): now also C8.1; no longer TP43.1
- new net: C10.2, C12.2
- new net: C11.1, TP44.1
- new net: C7.2, C8.2
- new net: C11.2, C9.2
- new net: C7.1, TP43.1
- new net: C12.1, TP45.1
Other:
- moved on the sheet: TP43, TP44, TP45

Commit message: Updated PCB
Parts:
- added H1, H2, H3, H4: MountingHole, MountingHole:MountingHole_3.2mm_M3, symbol Mechanical:MountingHole
- C6: footprint Capacitor_THT:CP_Radial_D4.0mm_P2.00mm -> Capacitor_THT:CP_Radial_D5.0mm_P2.00mm
- TP1, TP10, TP11, TP12, TP13, TP14, TP15, TP16, TP17, TP18, TP19, TP2, TP20, TP21, TP22, TP23, TP24, TP25, TP26, TP27, TP28, TP29, TP3, TP30, TP31, TP32, TP33, TP34, TP35, TP36, TP37, TP38, TP39, TP4, TP40, TP41, TP42, TP43, TP44, TP45, TP5, TP6, TP7, TP8, TP9: footprint TestPoint:TestPoint_THTPad_1.5x1.5mm_Drill0.7mm -> TestPoint:TestPoint_THTPad_2.0x2.0mm_Drill1.0mm
